File: EMB1/Sorter_Project01/PCB_LEDS/LED_board_2.brd (EAGLE design)
At the start: 100 x 80 mm, 10 parts, among them IC1 LM358N, K2 61201021621

Commit message: new boards
Connections:
- net GND: now also IC1.7
Routing:
- net GND: track 167.5 -> 170.1 mm
Changed lines of the file:
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@@
 <wire x1="43.688" y1="57.658" x2="45.974" y2="57.658" width="0.4064" layer="1"/>
 <wire x1="45.974" y1="57.658" x2="47.244" y2="56.388" width="0.4064" layer="1"/>
+<contactref element="IC1" pad="7"/>
+<wire x1="45.466" y1="14.986" x2="45.466" y2="12.446" width="0.6096" layer="1"/>
 </signal>
 <signal name="N$10">

Commit message: updated PCB design
Parts:
- moved R1 17.8 mm to (36.3, 22.6), turned to 180 degrees
Connections:
- net GND: now also IC1.3; no longer IC1.2
- net N$2: now also IC1.2; no longer IC1.3
Routing:
- net GND: track 170.1 -> 91.8 mm
- net PHD: track 97.1 -> 64.9 mm
- net N$2: track 58.3 -> 46.3 mm
Changed lines of the file:
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@@
 <layer number="17" name="Pads" color="2" fill="1" visible="yes" active="yes"/>
 <layer number="18" name="Vias" color="2" fill="1" visible="yes" active="yes"/>
-<layer number="19" name="Unrouted" color="6" fill="1" visible="yes" active="yes"/>
+<layer number="19" name="Unrouted" color="6" fill="1" visible="no" active="yes"/>
 <layer number="20" name="Dimension" color="15" fill="1" visible="yes" active="yes"/>
-<layer number="21" name="tPlace" color="7" fill="1" visible="yes" active="yes"/>
-<layer number="22" name="bPlace" color="7" fill="1" visible="yes" active="yes"/>
-<layer number="23" name="tOrigins" color="15" fill="1" visible="yes" active="yes"/>
-<layer number="24" name="bOrigins" color="15" fill="1" visible="yes" active="yes"/>
+<layer number="21" name="tPlace" color="7" fill="1" visible="no" active="yes"/>
+<layer number="22" name="bPlace" color="7" fill="1" visible="no" active="yes"/>
+<layer number="23" name="tOrigins" color="15" fill="1" visible="no" active="yes"/>
+<layer number="24" name="bOrigins" color="15" fill="1" visible="no" active="yes"/>
 <layer number="25" name="tNames" color="7" fill="1" visible="no" active="yes"/>
 <layer number="26" name="bNames" color="7" fill="1" visible="no" active="yes"/>
@@
 <element name="K2" library="Wurth_Elektronik_Electromechanic_Wire_to_Board_Connectors_rev15c" package="61201021621" value="61201021621" x="39.624" y="57.658"/>
 <element name="IC1" library="linear" package="DIL08" value="LM358N" x="41.656" y="13.716" rot="R270"/>
-<element name="R1" library="resistor" package="0207/10" value="" x="41.656" y="5.588"/>
+<element name="R1" library="resistor" package="0207/10" value="" x="36.322" y="22.606" rot="R180"/>
 </elements>
 <signals>
 <signal name="GND">
-<contactref element="OPTO" pad="A"/>
 <contactref element="K2" pad="9"/>
 <contactref element="IC1" pad="4"/>
-<contactref element="IC1" pad="2"/>
 <contactref element="IC1" pad="6"/>
 <contactref element="IC1" pad="5"/>
@@
 <contactref element="K2" pad="4"/>
 <contactref element="K2" pad="6"/>
-<wire x1="43.18" y1="40.64" x2="43.18" y2="41.148" width="0.6096" layer="1"/>
 <wire x1="43.18" y1="41.148" x2="44.958" y2="42.926" width="0.6096" layer="1"/>
 <wire x1="44.958" y1="42.926" x2="50.292" y2="42.926" width="0.6096" layer="1"/>
 <wire x1="50.292" y1="42.926" x2="51.562" y2="44.196" width="0.6096" layer="1"/>
 <wire x1="37.846" y1="9.906" x2="45.466" y2="9.906" width="0.6096" layer="1"/>
-<wire x1="37.846" y1="14.986" x2="37.338" y2="14.986" width="0.6096" layer="1"/>
-<wire x1="37.338" y1="14.986" x2="34.798" y2="12.446" width="0.6096" layer="1"/>
-<wire x1="34.798" y1="12.446" x2="34.798" y2="5.08" width="0.6096" layer="1"/>
-<wire x1="34.798" y1="5.08" x2="36.068" y2="3.81" width="0.6096" layer="1"/>
-<wire x1="36.068" y1="3.81" x2="39.37" y2="3.81" width="0.6096" layer="1"/>
-<wire x1="39.37" y1="3.81" x2="45.466" y2="9.906" width="0.6096" layer="1"/>
-<wire x1="37.846" y1="14.986" x2="39.37" y2="16.51" width="0.6096" layer="1"/>
-<wire x1="39.37" y1="16.51" x2="39.37" y2="21.844" width="0.6096" layer="1"/>
-<wire x1="39.37" y1="21.844" x2="36.322" y2="24.892" width="0.6096" layer="1"/>
-<wire x1="36.322" y1="24.892" x2="33.528" y2="24.892" width="0.6096" layer="1"/>
-<wire x1="33.528" y1="24.892" x2="27.432" y2="30.988" width="0.6096" layer="1"/>
-<wire x1="27.432" y1="30.988" x2="27.432" y2="49.276" width="0.6096" layer="1"/>
-<wire x1="27.432" y1="49.276" x2="37.084" y2="58.928" width="0.6096" layer="1"/>
 <wire x1="45.466" y1="12.446" x2="45.466" y2="9.906" width="0.6096" layer="1"/>
 <wire x1="47.244" y1="56.388" x2="51.562" y2="52.07" width="0.6096" layer="1"/>
@@
 <contactref element="IC1" pad="7"/>
 <wire x1="45.466" y1="14.986" x2="45.466" y2="12.446" width="0.6096" layer="1"/>
+<contactref element="OPTO" pad="A"/>
+<contactref element="IC1" pad="3"/>
+<wire x1="43.18" y1="41.148" x2="43.18" y2="40.64" width="0" layer="19" extent="1-1"/>
+<wire x1="37.846" y1="9.906" x2="37.846" y2="12.446" width="0.6096" layer="1"/>
 </signal>
 <signal name="N$10">
@@
 <wire x1="43.18" y1="32.004" x2="43.18" y2="33.02" width="0.6096" layer="1"/>
 </signal>
-<signal name="N$2">
-<contactref element="OPTO" pad="K"/>
-<contactref element="IC1" pad="3"/>
-<contactref element="R1" pad="1"/>
-<wire x1="40.64" y1="40.64" x2="40.64" y2="39.878" width="0.6096" layer="1"/>
-<wire x1="40.64" y1="39.878" x2="42.164" y2="38.354" width="0.6096" layer="1"/>
-<wire x1="42.164" y1="38.354" x2="43.688" y2="38.354" width="0.6096" layer="1"/>
-<wire x1="43.688" y1="38.354" x2="45.72" y2="40.386" width="0.6096" layer="1"/>
-<wire x1="45.72" y1="40.386" x2="51.308" y2="40.386" width="0.6096" layer="1"/>
-<wire x1="51.308" y1="40.386" x2="53.34" y2="38.354" width="0.6096" layer="1"/>
-<wire x1="53.34" y1="38.354" x2="53.34" y2="31.496" width="0.6096" layer="1"/>
-<wire x1="53.34" y1="31.496" x2="46.736" y2="24.892" width="0.6096" layer="1"/>
-<wire x1="40.64" y1="13.462" x2="39.624" y2="12.446" width="0.6096" layer="1"/>
-<wire x1="39.624" y1="12.446" x2="37.846" y2="12.446" width="0.6096" layer="1"/>
-<wire x1="40.64" y1="13.462" x2="40.64" y2="21.844" width="0.6096" layer="1"/>
-<wire x1="40.64" y1="21.844" x2="43.688" y2="24.892" width="0.6096" layer="1"/>
-<wire x1="43.688" y1="24.892" x2="46.736" y2="24.892" width="0.6096" layer="1"/>
-<wire x1="36.576" y1="5.588" x2="36.576" y2="11.176" width="0.6096" layer="1"/>
-<wire x1="36.576" y1="11.176" x2="37.846" y2="12.446" width="0.6096" layer="1"/>
-</signal>
 <signal name="PHD">
 <contactref element="R1" pad="2"/>
 <contactref element="IC1" pad="1"/>
 <contactref element="K2" pad="8"/>
-<wire x1="46.736" y1="5.588" x2="46.736" y2="4.826" width="0.6096" layer="1"/>
-<wire x1="46.736" y1="4.826" x2="44.196" y2="2.286" width="0.6096" layer="1"/>
-<wire x1="44.196" y1="2.286" x2="35.052" y2="2.286" width="0.6096" layer="1"/>
-<wire x1="35.052" y1="2.286" x2="33.02" y2="4.318" width="0.6096" layer="1"/>
-<wire x1="33.02" y1="4.318" x2="33.02" y2="14.224" width="0.6096" layer="1"/>
-<wire x1="33.02" y1="14.224" x2="36.322" y2="17.526" width="0.6096" layer="1"/>
-<wire x1="36.322" y1="17.526" x2="37.846" y2="17.526" width="0.6096" layer="1"/>
-<wire x1="37.846" y1="17.526" x2="37.846" y2="20.828" width="0.6096" layer="1"/>
-<wire x1="37.846" y1="20.828" x2="35.814" y2="22.86" width="0.6096" layer="1"/>
-<wire x1="35.814" y1="22.86" x2="33.02" y2="22.86" width="0.6096" layer="1"/>
-<wire x1="33.02" y1="22.86" x2="25.4" y2="30.48" width="0.6096" layer="1"/>
-<wire x1="25.4" y1="30.48" x2="25.4" y2="50.8" width="0.6096" layer="1"/>
 <wire x1="25.4" y1="50.8" x2="35.814" y2="61.214" width="0.6096" layer="1"/>
 <wire x1="35.814" y1="61.214" x2="42.418" y2="61.214" width="0.6096" layer="1"/>
 <wire x1="42.418" y1="61.214" x2="44.704" y2="58.928" width="0.6096" layer="1"/>
+<wire x1="25.4" y1="50.8" x2="25.4" y2="28.448" width="0.6096" layer="1"/>
+<wire x1="25.4" y1="28.448" x2="31.242" y2="22.606" width="0.6096" layer="1"/>
+<wire x1="31.242" y1="22.606" x2="31.242" y2="20.828" width="0.6096" layer="1"/>
+<wire x1="31.242" y1="20.828" x2="34.544" y2="17.526" width="0.6096" layer="1"/>
+<wire x1="34.544" y1="17.526" x2="37.846" y2="17.526" width="0.6096" layer="1"/>
 </signal>
 <signal name="5V">
@@
 <wire x1="53.086" y1="53.086" x2="47.244" y2="58.928" width="0.6096" layer="1"/>
 </signal>
+<signal name="N$2">
+<contactref element="IC1" pad="2"/>
+<contactref element="OPTO" pad="K"/>
+<contactref element="R1" pad="1"/>
+<wire x1="40.64" y1="40.64" x2="40.64" y2="39.37" width="0.6096" layer="1"/>
+<wire x1="40.64" y1="39.37" x2="41.148" y2="38.862" width="0.6096" layer="1"/>
+<wire x1="41.148" y1="38.862" x2="45.974" y2="38.862" width="0.6096" layer="1"/>
+<wire x1="45.974" y1="38.862" x2="46.736" y2="39.624" width="0.6096" layer="1"/>
+<wire x1="46.736" y1="39.624" x2="51.562" y2="39.624" width="0.6096" layer="1"/>
+<wire x1="51.562" y1="39.624" x2="53.34" y2="37.846" width="0.6096" layer="1"/>
+<wire x1="53.34" y1="37.846" x2="53.34" y2="32.004" width="0.6096" layer="1"/>
+<wire x1="53.34" y1="32.004" x2="46.228" y2="24.892" width="0.6096" layer="1"/>
+<wire x1="46.228" y1="24.892" x2="43.688" y2="24.892" width="0.6096" layer="1"/>
+<wire x1="41.402" y1="22.606" x2="43.688" y2="24.892" width="0.6096" layer="1"/>
+<wire x1="41.402" y1="22.606" x2="40.64" y2="21.844" width="0.6096" layer="1"/>
+<wire x1="40.64" y1="21.844" x2="40.64" y2="17.272" width="0.6096" layer="1"/>
+<wire x1="40.64" y1="17.272" x2="38.354" y2="14.986" width="0.6096" layer="1"/>
+<wire x1="38.354" y1="14.986" x2="37.846" y2="14.986" width="0.6096" layer="1"/>
+</signal>
 </signals>
