File: EMB1/FinalProject/schematics/Conectors_powersupply/Sch_PowerSupply.brd (EAGLE design)
At the start: 127 x 63.5 mm, 11 parts, among them IC2 LM2574N-3.3, K1 61201021621

Commit message: changes in pcb
Parts:
- removed K1: 61201021621, Wurth_Elektronik_Electromechanic_Wire_to_Board_Connectors_rev15c:61201021621
- added ENCODER1, ENCODER2: (no value), con-amp-quick:03P
- added SL2: (no value), con-amp-quick:02P
- moved D1 5.76 mm to (24.6, 26.4), turned to 270 degrees
- moved GYRO/ACC 0.25 mm to (52.1, 17.5)
Connections:
- removed net LBACK+: FPGA11/20.2, K1.5
- removed net LBACK-: FPGA11/20.1, K1.3
- removed net LFWD+: FPGA11/20.3, K1.7
- removed net LFWD-: FPGA1/10.10, K1.1
- removed net RBACK+: FPGA11/20.5, K1.6
- removed net RBACK-: FPGA11/20.6, K1.4
- removed net RFWD+: FPGA11/20.4, K1.8
- removed net RFWD-: FPGA11/20.7, K1.2
- new net N$11: FPGA1/10.9
- new net N$12: FPGA1/10.8
- new net N$7: FPGA11/20.3
- new net N$8: FPGA11/20.2
- new net SIGNAL1: ENCODER1.3, FPGA1/10.6
- new net SIGNAL2: ENCODER2.3, FPGA1/10.7
- net 3.3V: now also ENCODER1.1, ENCODER2.1
- net 5V: now also SL2.2
- net CL: now also FPGA11/20.4; no longer FPGA1/10.6
- net GND: now also ENCODER1.2, ENCODER2.2, SL2.1
- net MISO: now also FPGA11/20.5; no longer FPGA1/10.7
- net MOSI: now also FPGA11/20.7; no longer FPGA1/10.9
- net N$10: now also FPGA1/10.10; no longer K1.10
- net N$9: now also FPGA11/20.1; no longer K1.9
- net SCL: now also FPGA11/20.6; no longer FPGA1/10.8
Routing:
- net 3.3V: track 60.5 -> 108.6 mm
- net LFWD-: track 37.5 -> 0.00 mm
- net RFWD-: track 37.4 -> 0.00 mm
- net LBACK-: track 33.8 -> 0.00 mm
- net RBACK-: track 33.0 -> 0.00 mm
- net LBACK+: track 29.1 -> 0.00 mm
- net RBACK+: track 28.6 -> 0.00 mm
- net LFWD+: track 24.6 -> 0.00 mm
- net RFWD+: track 24.2 -> 0.00 mm
- net SIGNAL2: track 0.00 -> 17.0 mm
- net SIGNAL1: track 0.00 -> 15.2 mm
- net 5V: track 89.2 -> 103.6 mm
- net MOSI: track 32.9 -> 19.8 mm
- net SCL: track 32.8 -> 19.8 mm
- net MISO: track 32.4 -> 19.8 mm
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- removed copper zone on layer 16, net GND
